File: schematics/kiCad/blinky-brantevik.sch (KiCad schematic (older format))
At the start: 17 parts, among them J1 Screw_Terminal_01x03, J2 Screw_Terminal_01x03, J3 Screw_Terminal_01x04, J4 Screw_Terminal_01x02, U1 FEATHER_M0_BASIC_PROTO, U2 HC06

Commit message: more schem layout
Connections:
- no-connect marks 14 -> 15
Changed lines of the file:
@@
 NoConn ~ 4250 3400
 NoConn ~ 6650 3400
+NoConn ~ 4250 4900
 $EndSCHEMATC
