File: schematics/kiCad/blinky-brantevik.kicad_pcb (KiCad board)
At the start: 2 copper layers, 96 x 59 mm, 17 parts, among them J1 Screw_Terminal_01x03, J2 Screw_Terminal_01x03, J3 Screw_Terminal_01x04, J4 Screw_Terminal_01x02, U1 FEATHER_M0_BASIC_PROTO, U2 HC06

Commit message: more schem layout
Parts:
- moved R6 48.4 mm to (148.0, 123.5), turned to 270 degrees
- moved R7 46.5 mm to (135.5, 114.5), turned to 90 degrees
- moved C2 32.1 mm to (177.6, 119.5), turned to 180 degrees
- moved J4 30.5 mm to (108.0, 84.5), turned to 270 degrees
- moved R1 27.0 mm to (192.4, 117.0)
- moved J2 26.7 mm to (157.5, 84.0)
- moved D1 26.5 mm to (194.0, 111.5)
- moved D3 19.1 mm to (194.0, 87.0)
- moved R5 18.6 mm to (192.4, 93.0)
- moved R3 10.8 mm to (169.5, 99.5), turned to 90 degrees
- moved J1 6.02 mm to (157.5, 100.7)
- moved R4 5.32 mm to (169.5, 92.5), turned to 90 degrees
- moved R2 5.22 mm to (192.4, 105.5)
- moved D2 4.27 mm to (194.0, 99.5)
- moved J3 2.50 mm to (108.0, 100.5), turned to 270 degrees
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Connections:
- U1 pad P1_1: GND -> Net-(U1-PadP1_1)

Commit message: pcb complete
Parts:
- added Ant1: MountingHole_2.5mm, MountingHole:MountingHole_2.5mm, F.Cu at (180.6, 72.2)
- added G***: LOGO, dmcginnis427Footprints:blmcLogo, B.Cu at (134.0, 82.0)
- added G***: LOGO, dmcginnis427Footprints:blmcLogo, F.Cu at (134.0, 91.0)
- moved R7 42.5 mm to (177.9, 113.0), turned to 180 degrees
- moved R6 33.1 mm to (177.9, 109.5), turned to 180 degrees
- moved R3 15.4 mm to (157.4, 109.0), turned to 0 degrees
- moved R4 12.5 mm to (157.4, 89.0), turned to 0 degrees
- moved J1 3.34 mm to (157.5, 104.0)
- moved C2 1.12 mm to (176.6, 120.0)
Routing:
- net +5V: track 0.00 -> 134.1 mm, vias 0 -> 1
- net Net-(J3-Pad2): track 0.00 -> 119.2 mm, vias 0 -> 1
- net Net-(J3-Pad1): track 0.00 -> 90.3 mm, vias 0 -> 2
- net Net-(U1-PadP1_2): track 0.00 -> 58.3 mm, vias 0 -> 2
- net Net-(U1-PadP1_3): track 0.00 -> 54.9 mm, vias 0 -> 2
- net Net-(D3-Pad2): track 0.00 -> 28.2 mm
- net Net-(D2-Pad2): track 0.00 -> 28.2 mm
- net Net-(J1-Pad2): track 0.00 -> 22.2 mm
- net Net-(J1-Pad1): track 0.00 -> 17.1 mm
- net Net-(J2-Pad2): track 0.00 -> 16.5 mm
- net Net-(J2-Pad1): track 0.00 -> 14.7 mm
- net Net-(R6-Pad1): track 0.00 -> 8.34 mm
- net GND: track 0.00 -> 7.19 mm, vias 0 -> 16
- net Net-(D3-Pad1): track 0.00 -> 6.00 mm
- net Net-(D2-Pad1): track 0.00 -> 6.00 mm
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- added copper zone on B.Cu, net GND
- added copper zone on F.Cu, net GND
Other:
- outline, holes or cut-outs redrawn
- board text added: "Blinky-Brantevik-Cube V1.0"
